File: Hardware/Spectacle_LED_Control_Board.sch (EAGLE design)
At the start: 43 parts, among them J3 USB-MICROB, J4 AUDIO-JACK3, J8 AUDIO-JACK3, U1 CY8C4245LQI-483, U2 3.3V, U4 SN74LVC1G66, U5 SN74LVC1G66

Commit message: ready for review!
Other:
- note added: "03"
- note removed: "02"
Changed lines of the file:
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@@
 <wire x1="58.42" y1="86.36" x2="0" y2="86.36" width="0.3048" layer="97" style="longdash"/>
 <text x="165.1" y="7.62" size="2.54" layer="94" font="vector">Dia Campbell and Mike Hord</text>
-<text x="239.268" y="6.604" size="3.81" layer="91" font="vector">02</text>
+<text x="239.268" y="6.604" size="3.81" layer="91" font="vector">03</text>
 <wire x1="104.14" y1="127" x2="248.92" y2="127" width="0.3048" layer="97" style="longdash"/>
 <text x="236.22" y="129.54" size="3.81" layer="97" font="vector">MCU</text>
